File: OTTO-PCB/otto.brd (EAGLE design)
At the start: 57.2 x 53.3 mm, 16 parts, among them M1 ARDUINO-NANO-3.0, M2 SMALL_SERVO, M3 SMALL_SERVO, M4 SMALL_SERVO, M5 SMALL_SERVO

Commit message: Add files via upload
Parts:
- added C1, C3: 100nF, rcl:C025-025X050
- added R1, R2: 10K, rcl:0207/7
- C2: value (none) -> 47uF; device rcl:E15-5 -> rcl:140CLH-0810
- moved C2 6.48 mm to (45.7, 29.2), turned to 0 degrees
- moved M1 1.27 mm to (33.0, 27.9)
- moved JP6 0.63 mm to (57.8, 26.7), turned to 90 degrees
Connections:
- removed net N$28: M1.J2.5
- removed net RCK: JP6.3, M1.J1.15
- removed net SER: JP6.2, M1.J1.14
- new net CS: JP6.4, M1.J1.13
- new net DIN: JP6.2, M1.J1.15
- net +5V: now also C3.1, JP5.4, M1.J2.5
- net BUTTON1: now also R1.1
- net BUTTON2: now also R2.1
- net BUZZER: now also M1.J2.15; no longer M1.J1.13
- net CLK: now also JP6.3, M1.J1.14; no longer JP6.4, M1.J2.15
- net GND: now also C1.2, C3.2, R2.2; no longer JP5.4
- net NOISE: now also M1.J2.7; no longer M1.J2.6
- net V+: now also C1.1
Routing:
- net DIN: track 0.00 -> 52.5 mm
- net RCK: track 50.6 -> 0.00 mm
- net CS: track 0.00 -> 46.7 mm
- net SER: track 46.6 -> 0.00 mm
- net BUZZER: track 11.0 -> 25.0 mm
- net BUTTON1: track 12.0 -> 21.9 mm
- net BUTTON2: track 17.0 -> 20.8 mm
- net CLK: track 46.2 -> 49.9 mm
- net TX: track 48.9 -> 47.6 mm
- net TRIG: track 12.0 -> 13.2 mm
- net SERVO1: track 25.2 -> 23.9 mm
- net RX: track 48.9 -> 47.6 mm
- net ECHO: track 15.5 -> 16.5 mm
- net SERVO3: track 18.6 -> 18.1 mm
- net SERVO4: track 15.3 -> 14.8 mm
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Other:
- board text added: "+"
- board text added: "7219"
- board text added: "A5"
- board text added: "CS"
- board text added: "DIN"
- board text added: "S5"
- board text removed: "RCK"
- board text removed: "S1"
- board text removed: "SER"
