File: OTTO-PCB/otto.sch (EAGLE design)
At the start: 16 parts, among them M1 ARDUINO-NANO-3.0, M2 SMALL_SERVO, M3 SMALL_SERVO, M4 SMALL_SERVO, M5 SMALL_SERVO

Commit message: Add files via upload
Parts:
- added C1, C3: 100nF, rcl:C-EU025-025X050
- added R1, R2: 10K, rcl:R-EU_0207/7
- C2: value (none) -> 47uF; device rcl:CPOL-EUE15-5AXIAL -> rcl:CPOL-EU140CLH-0810
Connections:
- removed net N$28: M1.A7
- removed net RCK: JP6.3, M1.D12/MISO
- removed net SER: JP6.2, M1.D11/MOSI
- new net CS: JP6.4, M1.D10
- new net DIN: JP6.2, M1.D12/MISO
- net +5V: now also C3.1, JP5.4, M1.A7
- net BUTTON1: now also R1.1
- net BUTTON2: now also R2.1
- net BUZZER: now also M1.D13/SCK; no longer M1.D10
- net CLK: now also JP6.3, M1.D11/MOSI; no longer JP6.4, M1.D13/SCK
- net GND: now also C1.2, C3.2, R2.2; no longer JP5.4
- net NOISE: now also M1.A5; no longer M1.A6
- net V+: now also C1.1
Other:
- note added: "BUZZER PINS"
- note added: "MAX7219 LED matrix"
- note added: "PUSH BUTTONS"
- note added: "SOUND SENSOR PIN"
- note added: "ULTRASONIC MODULE"
